File: Resources-kopia/Templates/Kicad Templates/Easy-EMC Template/Easy-EMC.kicad_sch (KiCad schematic)
At the start: 6 parts, among them J1 GPIO, U1 CAT24C256

Commit message: upodate 3
Parts:
- removed C1: 100n, symbol Device:C_Small
- removed J1: GPIO, Connector_PinSocket_2.54mm:PinSocket_2x20_P2.54mm_Vertical, symbol Connector_Generic:Conn_02x20_Odd_Even
- removed JP1: ID_WP, symbol Jumper:SolderJumper_2_Open
- removed R1, R2: 3.9k, symbol Device:R_Small
- removed U1: CAT24C256, symbol Memory_EEPROM:CAT24C256
Connections:
- no-connect marks 3 -> 0
Other:
- note added: "Project Motor"
- note removed: "Additional pin functions: https://pinout.xyz/"
- note removed: "ID_SD and ID_SC PINS: These pins are reserved for HAT ID EEPROM. At boot time this I2C interface will be interrogated to look for an EEPROM that identifes the attached board and allows automagic setup of the GPIOs (and optionally, Linux drivers). Bridging JP1 enables write protection. DO NOT USE these pins for anything other than attaching an I2C ID EEPROM. Leave unconnected if ID EEPROM not requ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"
- company: (none) -> Company: Easy EMC
- title: (none) -> Project name: Project Motor
